File: PCB/main/usb.kicad_sch (KiCad schematic)
At the start: 5 parts, among them J1 TYPE-C-31-M-12, U8 USBLC6-2SC6, U9 PESD5V0S2BT,215

Commit message: fab: regenerate JLCPCB assembly/fab outputs for the routed board
- Complete the missing Manufacturer fields (verified against the live LCSC/JLC
  library) on the affected symbols and footprints; no connectivity, geometry,
  routing or value changes.
- Regenerate dist/jlcpcb: bom.csv, pick_and_place.csv, gerber.zip, export-report.json
  from the current board (export.py --overwrite --side top --require-part-numbers).
- BOM: R23 removed, R24/R25 added, TH1 (TDK NTCG103JF103FT1 / C209959) added,
  U4 corrected to XC6220B331MR-G / C86534.
- CPL: R23 row gone; R24, R25 and TH1 rows added.
- DRC: 0 violations, 0 unrouted; one schematic-parity warning (U4 symbol Footprint
  field reads SOT-23-5 while the board uses the identical-land SOT-25_XC6220).
Parts:
- J1: Manufacturer (none) -> Korean Hroparts Elec
- R1, R2: Manufacturer (none) -> UNI-ROYAL(Uniroyal Elec)
- U8: Manufacturer (none) -> STMicroelectronics
- U9: Manufacturer (none) -> Nexperia
Changed lines of the file:
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@@
+          (size 1 1))
+        (hide yes)))
+(property "Manufacturer" "Korean Hroparts Elec"
+      (at 78.74 92.71 0)
+      (effects
+        (font
           (size 1 1))
         (hide yes)))
@@
           (size 1 1))
         (hide yes)))
+(property "Manufacturer" "STMicroelectronics"
+      (at 149.86 82.55 0)
+      (effects
+        (font
+          (size 1 1))
+        (hide yes)))
     (pin "1"
 )
@@
           (size 1 1))
         (hide yes)))
+(property "Manufacturer" "Nexperia"
+      (at 149.86 128.27 0)
+      (effects
+        (font
+          (size 1 1))
+        (hide yes)))
     (pin "1"
 )
@@
           (size 1 1))
         (hide yes)))
+(property "Manufacturer" "UNI-ROYAL(Uniroyal Elec)"
+      (at 119.38 142.24 0)
+      (effects
+        (font
+          (size 1 1))
+        (hide yes)))
     (pin "1"
 )
@@
       (at 106.68 152.4 0)
       (effects
+        (font
+          (size 1 1))
+        (hide yes)))
+(property "Manufacturer" "UNI-ROYAL(Uniroyal Elec)"
+      (at 106.68 152.4 0)
+      (effects
