File: PCB/main/power.kicad_sch (KiCad schematic)
At the start: 16 parts, among them J2 Battery wire pads 2.54mm, SW1 Off-board pack toggle switch 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, U4 XC6220B331MR-G, U6 BQ24074RGTR

Commit message: power: add pack-NTC cell-temperature sensing on charger TS (Option A)
- J2 becomes a 3-contact pack pad group (BAT+ / BAT- / NTC): new symbol + new footprint BatteryWire_3x_PTH_P2.54mm_D1.0mm (pad 3 added 2.54mm beyond pad 2, existing pads 1/2 unchanged)
- TS (U6 pin 1) now senses the in-pack 10k B3435 NTC (TH1, off-board, in_bom no) instead of the 10k fixed bias; charger suspends ~0..51C natively
- R23 (10k TS bias) set DNP / in_bom no - fallback for 2-wire packs only; must NOT be fitted with an NTC pack
- Annotations updated. Schematic-only ECO: layout/routing/footprint placement intentionally not updated
Parts:
- added TH1: 10k B3435 NTC (in-pack, cell-bonded, off-board), symbol Device:Thermistor_NTC
- J2: value Battery wire pads 2.54mm -> Battery wire pads 3x 2.54mm; footprint smove-r2-main:BatteryWire_2x_PTH_P2.54mm_D1.0mm -> smove-r2-main:BatteryWire_3x_PTH_P2.54mm_D1.0mm; symbol smove-r2-main:J2 -> smove-r2-main:BatteryWire_3x_PTH_P2.54mm_D1.0mm
- R23: now not fitted; now left out of the parts list
Connections:
- net GND: now also TH1.2
- net TS_NO_CELL_SENSING renamed TS
- net TS: now also J2.3 (NTC), TH1.1
Other:
- note added: "Cell sensing: TS = 10k NTC in pack (J2 pin NTC, beta ~3435). R23 DNP (2-wire pack fallback). TMR / ITERM open; CE / EN2 grounded; EN1 pulled up to SYS = USB500. No source/CC awareness."
- note added: "J2 3x pads = 1 BAT+ / 2 BAT- / 3 NTC (10k B3435 cell-bonded, 103AT-2 class): charger suspends outside ~0C..50C (TS 300mV/2.1V). Do NOT fit R23 with an NTC pack."
- note added: "USB500 input-current limit ~500mA (450mA guaranteed-min): EN1 pulled up to SYS. Protected 4.2V pack only. Cell-temperature sensing: 10k NTC in pack on U6 TS (J2 pin 3)."
- note removed: "NO cell sensing: TS 10k bias. TMR / ITERM open; CE / EN2 grounded; EN1 pulled up to SYS = USB500. No source/CC awareness."
- note removed: "USB500 input-current limit ~500mA (450mA guaranteed-min): EN1 pulled up to SYS. Protected 4.2V pack only. No automatic cell-temperature sensing."
Changed lines of the file:
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@@
           (unit 1)))))
   (symbol
-    (lib_id "smove-r2-main:J2")
+    (lib_id "smove-r2-main:BatteryWire_3x_PTH_P2.54mm_D1.0mm")
     (at 50.8 87.63 0)
     (unit 1)
@@
         (font
           (size 1 1))))
-    (property "Value" "Battery wire pads 2.54mm"
+    (property "Value" "Battery wire pads 3x 2.54mm"
       (at 25.4 87.376 0)
       (effects
         (font
           (size 0.95 0.95))))
-    (property "Footprint" "smove-r2-main:BatteryWire_2x_PTH_P2.54mm_D1.0mm"
+    (property "Footprint" "smove-r2-main:BatteryWire_3x_PTH_P2.54mm_D1.0mm"
       (at 50.8 77.47 0)
       (effects
@@
     (pin "2"
 )
+    (pin "3"
+)
     (instances
       (project "smove-r2-main"
         (path "/8e261347-838a-5848-981d-f693675e8aa0/a926f61e-132d-5af0-876e-12788077b17d"
           (reference "J2")
+          (unit 1)))))
+  (symbol
+    (lib_id "Device:Thermistor_NTC")
+    (at 60.96 121.92 0)
+    (unit 1)
+    (in_bom no)
+    (on_board no)
+    (dnp no)
+    (property "Reference" "TH1"
+      (at 56.896 120.269 0)
+      (effects
+        (font
+          (size 0.95 0.95))
+        (justify right)))
+    (property "Value" "10k B3435 NTC (in-pack, cell-bonded, off-board)"
+      (at 56.896 123.571 0)
+      (effects
+        (font
+          (size 0.9 0.9))
+        (justify right)))
+    (property "Footprint" ""
+      (at 60.96 121.92 0)
+      (effects
+        (font
+          (size 1 1))
+        (hide yes)))
+    (property "MPN" "103AT-2"
+      (at 60.96 121.92 0)
+      (effects
+        (font
+          (size 1 1))
+        (hide yes)))
+    (property "LCSC" ""
+      (at 60.96 121.92 0)
+      (effects
+        (font
+          (size 1 1))
+        (hide yes)))
+    (property "Description" "Off-board, cell-bonded pack thermistor (not on this PCB). Semitec 103AT-2 class: R25 = 10k, B25/85 = 3435 K. Wired TS -> pack BAT- (J2 pin 3 -> pin 2). Charger TS window ~0 C .. 51 C (TI SLUS810N sec. 8.5 / 9.3.6)."
+      (at 60.96 121.92 0)
+      (effects
+        (font
+          (size 1 1))
+        (hide yes)))
+    (pin "1"
+)
+    (pin "2"
+)
+    (instances
+      (project "smove-r2-main"
+        (path "/8e261347-838a-5848-981d-f693675e8aa0/a926f61e-132d-5af0-876e-12788077b17d"
+          (reference "TH1")
+          (unit 1)))))
+  (symbol
+    (lib_id "power:GND")
+    (at 60.96 128.27 0)
+    (unit 1)
+    (in_bom no)
+    (on_board no)
+    (dnp no)
+    (property "Reference" "#PWR27"
+      (at 60.96 120.65 0)
+      (effects
+        (font
+          (size 1 1))
+        (hide yes)))
+    (property "Value" "GND"
+      (at 60.96 124.206 0)
+      (effects
+        (font
+          (size 0.95 0.95))
+        (hide yes)))
+    (pin "1"
+)
+    (instances
+      (project "smove-r2-main"
+        (path "/8e261347-838a-5848-981d-f693675e8aa0/a926f61e-132d-5af0-876e-12788077b17d"
+          (reference "#PWR27")
           (unit 1)))))
   (symbol
@@
     (at 71.12 134.62 0)
     (unit 1)
-    (in_bom yes)
+    (in_bom no)
     (on_board yes)
-    (dnp no)
+    (dnp yes)
     (property "Reference" "R23"
       (at 79.248 132.969 0)
@@
         (path "/8e261347-838a-5848-981d-f693675e8aa0/a926f61e-132d-5af0-876e-12788077b17d"
           (reference "R23")
-          (unit 1)))))
+          (unit 1))))
+    (property "Description" "DNP: 10k TS-to-VSS bias for 2-wire packs without an in-pack NTC (charger TS function unused, therefore no cell-temperature protection). Must NOT be fitted when the pack NTC is wired to J2 pin 3."
+      (at 71.12 134.62 0)
+      (effects
+        (font
+          (size 1 1))
+        (hide yes))))
   (symbol
     (lib_id "Device:C")
@@
       (justify left bottom))
 )
-  (label "TS_NO_CELL_SENSING"
+  (label "TS"
     (at 71.12 91.44 0)
     (effects
@@
       (justify left bottom))
 )
-  (text "USB500 input-current limit ~500mA (450mA guaranteed-min): EN1 pulled up to SYS. Protected 4.2V pack only. No automatic cell-temperature sensing."
+  (label "TS"
+    (at 60.96 99.06 90)
+    (effects
+      (font
+        (size .85 .85))
+      (justify left bottom))
+)
+  (text "USB500 input-current limit ~500mA (450mA guaranteed-min): EN1 pulled up to SYS. Protected 4.2V pack only. Cell-temperature sensing: 10k NTC in pack on U6 TS (J2 pin 3)."
     (at 25.4 24.13 0)
     (effects
@@
       (justify left))
 )
-  (text "NO cell sensing: TS 10k bias. TMR / ITERM open; CE / EN2 grounded; EN1 pulled up to SYS = USB500. No source/CC awareness."
+  (text "Cell sensing: TS = 10k NTC in pack (J2 pin NTC, beta ~3435). R23 DNP (2-wire pack fallback). TMR / ITERM open; CE / EN2 grounded; EN1 pulled up to SYS = USB500. No source/CC awareness."
     (at 25.4 170.18 0)
+    (effects
+      (font
+        (size 0.9 0.9))
+      (justify left))
+)
+  (text "J2 3x pads = 1 BAT+ / 2 BAT- / 3 NTC (10k B3435 cell-bonded, 103AT-2 class): charger suspends outside ~0C..50C (TS 300mV/2.1V). Do NOT fit R23 with an NTC pack."
+    (at 25.4 173.99 0)
     (effects
       (font
@@
     (stroke
       (width 0)
+      (type default))
+)
+  (wire
+    (pts
+      (xy 60.96 96.52)
+      (xy 60.96 118.11))
+    (stroke
+      (width 0)
+      (type default))
+)
+  (wire
+    (pts
+      (xy 60.96 125.73)
+      (xy 60.96 128.27))
+    (stroke
+      (width 0)

Commit message: power: separate on-board NTC part, drawn TS/SYS nets, drop R23 and J2 NTC contact
- J2 restored to the 2-contact pack connector (BAT+ / BAT-); the NTC contact is gone.
- TH1 is now its own part: project symbol smove-r2-main:NTC_10K_B3435 + project footprint
  smove-r2-main:NTC_0402_1005Metric (TDK NTCG103JF103FT1, LCSC C209959), in_bom/on_board yes,
  wired directly U6.1 (TS) -> TH1.1 and TH1.2 -> GND.
- TS and SYS nets are now single continuous drawn wires (one label each kept for net naming);
  the label-only joins are gone, and the dangling TS stub is removed.
- R23 deleted outright (symbol, wires, orphaned #PWR19 GND symbol, all sheet text references).
- BatteryWire_3x_PTH_P2.54mm_D1.0mm symbol + footprint removed as dead library clutter.
- Schematic-only ECO: PCB/layout, other sheets, lib tables and dist/ intentionally untouched.
Parts:
- removed R23: 10k, smove-r2-main:R_0402_1005Metric, symbol Device:R
- J2: value Battery wire pads 3x 2.54mm -> Battery wire pads 2x 2.54mm; footprint smove-r2-main:BatteryWire_3x_PTH_P2.54mm_D1.0mm -> smove-r2-main:BatteryWire_2x_PTH_P2.54mm_D1.0mm; symbol smove-r2-main:BatteryWire_3x_PTH_P2.54mm_D1.0mm -> smove-r2-main:BatteryWire_2x_PTH_P2.54mm_D1.0mm
- TH1: value 10k B3435 NTC (in-pack, cell-bonded, off-board) -> 10k B3435 NTC (cell-bonded); footprint (none) -> smove-r2-main:NTC_0402_1005Metric; symbol Device:Thermistor_NTC -> smove-r2-main:NTC_10K_B3435; LCSC (none) -> C209959; MPN 103AT-2 -> NTCG103JF103FT1; now in the parts list
Connections:
- net TS: no longer J2.3 (NTC)
Other:
- note added: "Cell sensing: TS = TH1, a separate on-board 10k B3435 NTC (0402) wired directly TS -> GND. An open NTC lead floats TS high and inhibits charging. TMR / ITERM open; CE / EN2 grounded; EN1 pulled up to SYS = USB500. No source/CC awareness."
- note added: "J2 = 2-contact pack connector (BAT+ / BAT- only). The cell thermistor is not routed through the pack harness: TH1 is a separate on-board part. Charger suspends outside ~0C..50C (TS 300mV/2.1V)."
- note added: "USB500 input-current limit ~500mA (450mA guaranteed-min): EN1 pulled up to SYS. Protected 4.2V pack only. Cell-temperature sensing: on-board TH1 (10k B3435 NTC, 0402, cell-bonded) on U6 TS."
- note removed: "Cell sensing: TS = 10k NTC in pack (J2 pin NTC, beta ~3435). R23 DNP (2-wire pack fallback). TMR / ITERM open; CE / EN2 grounded; EN1 pulled up to SYS = USB500. No source/CC awareness."
- note removed: "J2 3x pads = 1 BAT+ / 2 BAT- / 3 NTC (10k B3435 cell-bonded, 103AT-2 class): charger suspends outside ~0C..50C (TS 300mV/2.1V). Do NOT fit R23 with an NTC pack."
- note removed: "USB500 input-current limit ~500mA (450mA guaranteed-min): EN1 pulled up to SYS. Protected 4.2V pack only. Cell-temperature sensing: 10k NTC in pack on U6 TS (J2 pin 3)."

Commit message: fab: regenerate JLCPCB assembly/fab outputs for the routed board
- Complete the missing Manufacturer fields (verified against the live LCSC/JLC
  library) on the affected symbols and footprints; no connectivity, geometry,
  routing or value changes.
- Regenerate dist/jlcpcb: bom.csv, pick_and_place.csv, gerber.zip, export-report.json
  from the current board (export.py --overwrite --side top --require-part-numbers).
- BOM: R23 removed, R24/R25 added, TH1 (TDK NTCG103JF103FT1 / C209959) added,
  U4 corrected to XC6220B331MR-G / C86534.
- CPL: R23 row gone; R24, R25 and TH1 rows added.
- DRC: 0 violations, 0 unrouted; one schematic-parity warning (U4 symbol Footprint
  field reads SOT-23-5 while the board uses the identical-land SOT-25_XC6220).
Parts:
- C1, C11, C13, C2, C3: Manufacturer (none) -> Samsung Electro-Mechanics
- R14, R15, R21, R22, R24, R25: Manufacturer (none) -> UNI-ROYAL(Uniroyal Elec)
- TH1: Manufacturer (none) -> TDK
- U4: Manufacturer (none) -> Torex Semicon
- U6: Manufacturer (none) -> Texas Instruments
Changed lines of the file:
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@@
+          (size 1 1))
+        (hide yes)))
+(property "Manufacturer" "Texas Instruments"
+      (at 106.68 71.12 0)
+      (effects
+        (font
           (size 1 1))
         (hide yes)))
@@
         (hide yes)))
     (property "LCSC" "C86534"
+      (at 187.96 50.8 0)
+      (effects
+        (font
+          (size 1 1))
+        (hide yes)))
+(property "Manufacturer" "Torex Semicon"
       (at 187.96 50.8 0)
       (effects
@@
           (size 1 1))
         (hide yes)))
+(property "Manufacturer" "TDK"
+      (at 60.96 121.92 0)
+      (effects
+        (font
+          (size 1 1))
+        (hide yes)))
     (property "Description" "On-board 0402 cell thermistor on the BQ24074 TS pin: TS (U6.1) -> TH1.1, TH1.2 -> GND. Sets the charger temperature window ~0 C .. 50 C (TS 300mV / 2.1V); charging is inhibited outside it, and an open NTC lead floats TS high and also inhibits charging. Cell-bonded placement, 10k B3435."
       (at 60.96 121.92 0)
@@
           (size 1 1))
         (hide yes)))
+(property "Manufacturer" "UNI-ROYAL(Uniroyal Elec)"
+      (at 157.48 121.92 0)
+      (effects
+        (font
+          (size 1 1))
+        (hide yes)))
     (pin "1"
 )
@@
           (size 1 1))
         (hide yes)))
+(property "Manufacturer" "UNI-ROYAL(Uniroyal Elec)"
+      (at 157.48 142.24 0)
+      (effects
+        (font
+          (size 1 1))
+        (hide yes)))
     (pin "1"
 )
@@
           (size 1 1))
         (hide yes)))
+(property "Manufacturer" "UNI-ROYAL(Uniroyal Elec)"
+      (at 144.78 119.38 0)
+      (effects
+        (font
+          (size 1 1))
+        (hide yes)))
     (pin "1"
 )
@@
           (size 1 1))
         (hide yes)))
+(property "Manufacturer" "UNI-ROYAL(Uniroyal Elec)"
+      (at 129.54 137.16 0)
+      (effects
+        (font
+          (size 1 1))
+        (hide yes)))
     (pin "1"
 )
@@
           (size 1 1))
         (hide yes)))
+(property "Manufacturer" "Samsung Electro-Mechanics"
+      (at 48.26 50.8 0)
+      (effects
+        (font
+          (size 1 1))
+        (hide yes)))
     (pin "1"
 )
@@
           (size 1 1))
         (hide yes)))
+(property "Manufacturer" "Samsung Electro-Mechanics"
+      (at 63.5 101.6 0)
+      (effects
+        (font
+          (size 1 1))
+        (hide yes)))
     (pin "1"
 )
@@
           (size 1 1))
         (hide yes)))
+(property "Manufacturer" "Samsung Electro-Mechanics"
+      (at 205.74 63.5 0)
+      (effects
+        (font
+          (size 1 1))
+        (hide yes)))
     (pin "1"
 )
@@
           (size 1 1))
         (hide yes)))
+(property "Manufacturer" "Samsung Electro-Mechanics"
+      (at 177.8 142.24 0)
+      (effects
+        (font
+          (size 1 1))
+        (hide yes)))
     (pin "1"
 )
@@
         (hide yes)))
     (property "LCSC" "C16780"
+      (at 160.02 60.96 0)
+      (effects
+        (font
+          (size 1 1))
+        (hide yes)))
+(property "Manufacturer" "Samsung Electro-Mechanics"
       (at 160.02 60.96 0)
       (effects
@@
           (size 1 1))
         (hide yes)))
+(property "Manufacturer" "UNI-ROYAL(Uniroyal Elec)"
+      (at 66.04 52.07 0)
+      (effects
+        (font
+          (size 1 1))
+        (hide yes)))
     (pin "1"
 )
@@
       (at 134.62 111.76 0)
       (effects
+        (font
+          (size 1 1))
+        (hide yes)))
+(property "Manufacturer" "UNI-ROYAL(Uniroyal Elec)"
+      (at 134.62 111.76 0)
+      (effects
